Commit message: Add initial modality probe instrumentation

File: models/rotors_description/urdf/component_snippets.xacro (robot description, xacro)
@@ -201,4 +201,12 @@
     <gazebo>
       <plugin name='groundtruth_plugin' filename='libgazebo_groundtruth_plugin.so'>
+        <robotNamespace>${namespace}</robotNamespace>
+      </plugin>
+    </gazebo>
+  </xacro:macro>
+  <!-- Macro to add the Modality probe plugin. -->
+  <xacro:macro name="probe_plugin_macro" params="namespace">
+    <gazebo>
+      <plugin name='probe_plugin' filename='libgazebo_probe_plugin.so'>
         <robotNamespace>${namespace}</robotNamespace>
       </plugin>

File: models/rotors_description/urdf/iris_base.xacro (robot description, xacro)
@@ -53,5 +53,5 @@
   <xacro:arg name='use_tcp' default='true' />
   <xacro:arg name='vehicle_is_tailsitter' default='false' />
-  <xacro:arg name='visual_material' default='DarkGrey' />
+  <xacro:arg name='visual_material' default='Orange' />
   <xacro:arg name='enable_mavlink_interface' default='true' />
   <xacro:arg name='enable_wind' default='false' />
@@ -60,4 +60,5 @@
   <xacro:arg name='enable_logging' default='false' />
   <xacro:arg name='log_file' default='iris' />
+  <xacro:arg name='enable_probe' default='false' />
   <!-- macros for gazebo plugins, sensors -->
   <xacro:include filename="$(arg rotors_description_dir)/urdf/component_snippets.xacro" />
@@ -97,4 +98,9 @@
     >
   </xacro:groundtruth_plugin_macro>
+  <!-- Instantiate Modality probe plugin. -->
+  <xacro:probe_plugin_macro
+    namespace="${namespace}"
+    >
+  </xacro:probe_plugin_macro>
   <!-- Instantiate magnetometer plugin. -->
   <xacro:magnetometer_plugin_macro
